Commit message: Stage 7A: add simulated 2D lidar (LaserScan)
The nori_hardware plugin casts a mj_ray fan from a new 'lidar' MJCF site each
control cycle and publishes sensor_msgs/LaserScan on /scan (throttled, default
360 beams @ 10 Hz). Rays are masked to geom group 2 so the beam sees the
mappable environment, not the robot's own body.

- simulation/mujoco/nori.xml: lidar mount site on the base
- simulation/mujoco/scene.xml: 6x6 m room + obstacle (group 2) to scan
- ros/nori_description: lidar_link TF frame matching the MJCF site
- ros/nori_hardware: LaserScan publisher, sensor_msgs dep
- ros/test_lidar.sh + _check_lidar.py: gate (scan sane, in-room, TF present)
- docs/PLAN.md: north star (dishes->rack->dishwasher) + 7A-7F milestone ladder

File: ros/nori_description/urdf/nori.urdf.xacro (robot description, xacro)
@@ -26,4 +26,14 @@
   <xacro:wheel side="left"  y="0.13"/>
   <xacro:wheel side="right" y="-0.13"/>
+  <!-- 2D lidar frame — matches the "lidar" site in simulation/mujoco/nori.xml.
+       The nori_hardware plugin publishes /scan in this frame. -->
+  <link name="lidar_link">
+    <visual><geometry><cylinder radius="0.03" length="0.04"/></geometry>
+      <material name="dark"/></visual>
+  </link>
+  <joint name="lidar_joint" type="fixed">
+    <parent link="base_link"/><child link="lidar_link"/>
+    <origin xyz="0.12 0 0.19"/>
+  </joint>
   <!-- torso lift (prismatic) -->
   <link name="torso_link">
